Commit message: Fix gz-sim joint control on both robots and add H1 lidar SLAM plus pretrained RL walk

File: ros2_ws/src/h1_description/urdf/h1.urdf (robot description, URDF)
Before this commit: robot h1_description, 25 links, 24 joints
Links:
- link left_ankle_link: geometry collision box size=0.28 0.10 0.024; visual mesh filename=package://h1_description/meshes/left_ankle_link.STL
- link right_ankle_link: geometry collision box size=0.28 0.10 0.024; visual mesh filename=package://h1_description/meshes/right_ankle_link.STL
